Commit message: Update for simulation

File: urdf/TankBot.xacro (robot description, xacro)
@@ -1,7 +1,7 @@
 <?xml version="1.0" ?>
 <robot name="TankBot" xmlns:xacro="http://www.ros.org/wiki/xacro">
-<xacro:include filename="$(find TankBot_description)/urdf/materials.xacro" />
-<xacro:include filename="$(find TankBot_description)/urdf/TankBot.trans" />
-<xacro:include filename="$(find TankBot_description)/urdf/TankBot.gazebo" />
+<xacro:include filename="$(find tankbot_description)/urdf/materials.xacro" />
+<xacro:include filename="$(find tankbot_description)/urdf/TankBot.trans" />
+<xacro:include filename="$(find tankbot_description)/urdf/TankBot.gazebo" />
 <link name="base_link">
   <inertial>
@@ -13,5 +13,5 @@
     <origin xyz="0 0 0" rpy="0 0 0"/>
     <geometry>
-      <mesh filename="file://$(find TankBot_description)/meshes/base_link.stl" scale="0.001 0.001 0.001"/>
+      <mesh filename="file://$(find tankbot_description)/meshes/base_link.stl" scale="0.001 0.001 0.001"/>
     </geometry>
     <material name="silver"/>
@@ -20,5 +20,5 @@
     <origin xyz="0 0 0" rpy="0 0 0"/>
     <geometry>
-      <mesh filename="file://$(find TankBot_description)/meshes/base_link.stl" scale="0.001 0.001 0.001"/>
+      <mesh filename="file://$(find tankbot_description)/meshes/base_link.stl" scale="0.001 0.001 0.001"/>
     </geometry>
   </collision>
@@ -33,5 +33,5 @@
     <origin xyz="0.117325 0.102175 0.033" rpy="0 0 0"/>
     <geometry>
-      <mesh filename="file://$(find TankBot_description)/meshes/roda_dentada_v2_1.stl" scale="0.001 0.001 0.001"/>
+      <mesh filename="file://$(find tankbot_description)/meshes/roda_dentada_v2_1.stl" scale="0.001 0.001 0.001"/>
     </geometry>
     <material name="silver"/>
@@ -40,5 +40,5 @@
     <origin xyz="0.117325 0.102175 0.033" rpy="0 0 0"/>
     <geometry>
-      <mesh filename="file://$(find TankBot_description)/meshes/roda_dentada_v2_1.stl" scale="0.001 0.001 0.001"/>
+      <mesh filename="file://$(find tankbot_description)/meshes/roda_dentada_v2_1.stl" scale="0.001 0.001 0.001"/>
     </geometry>
   </collision>
@@ -53,5 +53,5 @@
     <origin xyz="0.067305 0.104175 0.069726" rpy="0 0 0"/>
     <geometry>
-      <mesh filename="file://$(find TankBot_description)/meshes/roda_lisa_v2__2__1.stl" scale="0.001 0.001 0.001"/>
+      <mesh filename="file://$(find tankbot_description)/meshes/roda_lisa_v2__2__1.stl" scale="0.001 0.001 0.001"/>
     </geometry>
     <material name="silver"/>
@@ -60,5 +60,5 @@
     <origin xyz="0.067305 0.104175 0.069726" rpy="0 0 0"/>
     <geometry>
-      <mesh filename="file://$(find TankBot_description)/meshes/roda_lisa_v2__2__1.stl" scale="0.001 0.001 0.001"/>
+      <mesh filename="file://$(find tankbot_description)/meshes/roda_lisa_v2__2__1.stl" scale="0.001 0.001 0.001"/>
     </geometry>
   </collision>
@@ -73,5 +73,5 @@
     <origin xyz="0.022305 0.104175 0.069726" rpy="0 0 0"/>
     <geometry>
-      <mesh filename="file://$(find TankBot_description)/meshes/roda_lisa_v2__3__1.stl" scale="0.001 0.001 0.001"/>
+      <mesh filename="file://$(find tankbot_description)/meshes/roda_lisa_v2__3__1.stl" scale="0.001 0.001 0.001"/>
     </geometry>
     <material name="silver"/>
@@ -80,5 +80,5 @@
     <origin xyz="0.022305 0.104175 0.069726" rpy="0 0 0"/>
     <geometry>
-      <mesh filename="file://$(find TankBot_description)/meshes/roda_lisa_v2__3__1.stl" scale="0.001 0.001 0.001"/>
+      <mesh filename="file://$(find tankbot_description)/meshes/roda_lisa_v2__3__1.stl" scale="0.001 0.001 0.001"/>
     </geometry>
   </collision>
@@ -93,5 +93,5 @@
     <origin xyz="-0.022695 0.104175 0.069726" rpy="0 0 0"/>
     <geometry>
-      <mesh filename="file://$(find TankBot_description)/meshes/roda_lisa_v2__4__1.stl" scale="0.001 0.001 0.001"/>
+      <mesh filename="file://$(find tankbot_description)/meshes/roda_lisa_v2__4__1.stl" scale="0.001 0.001 0.001"/>
     </geometry>
     <material name="silver"/>
@@ -100,5 +100,5 @@
     <origin xyz="-0.022695 0.104175 0.069726" rpy="0 0 0"/>
     <geometry>
-      <mesh filename="file://$(find TankBot_description)/meshes/roda_lisa_v2__4__1.stl" scale="0.001 0.001 0.001"/>
+      <mesh filename="file://$(find tankbot_description)/meshes/roda_lisa_v2__4__1.stl" scale="0.001 0.001 0.001"/>
     </geometry>
   </collision>
@@ -113,5 +113,5 @@
     <origin xyz="-0.069695 0.104175 0.069726" rpy="0 0 0"/>
     <geometry>
-      <mesh filename="file://$(find TankBot_description)/meshes/roda_lisa_v2__5__1.stl" scale="0.001 0.001 0.001"/>
+      <mesh filename="file://$(find tankbot_description)/meshes/roda_lisa_v2__5__1.stl" scale="0.001 0.001 0.001"/>
     </geometry>
     <material name="silver"/>
@@ -120,5 +120,5 @@
     <origin xyz="-0.069695 0.104175 0.069726" rpy="0 0 0"/>
     <geometry>
-      <mesh filename="file://$(find TankBot_description)/meshes/roda_lisa_v2__5__1.stl" scale="0.001 0.001 0.001"/>
+      <mesh filename="file://$(find tankbot_description)/meshes/roda_lisa_v2__5__1.stl" scale="0.001 0.001 0.001"/>
     </geometry>
   </collision>
@@ -133,5 +133,5 @@
     <origin xyz="-0.120175 0.102175 0.033" rpy="0 0 0"/>
     <geometry>
-      <mesh filename="file://$(find TankBot_description)/meshes/roda_lisa_v2__6__1.stl" scale="0.001 0.001 0.001"/>
+      <mesh filename="file://$(find tankbot_description)/meshes/roda_lisa_v2__6__1.stl" scale="0.001 0.001 0.001"/>
     </geometry>
     <material name="silver"/>
@@ -140,5 +140,5 @@
     <origin xyz="-0.120175 0.102175 0.033" rpy="0 0 0"/>
     <geometry>
-      <mesh filename="file://$(find TankBot_description)/meshes/roda_lisa_v2__6__1.stl" scale="0.001 0.001 0.001"/>
+      <mesh filename="file://$(find tankbot_description)/meshes/roda_lisa_v2__6__1.stl" scale="0.001 0.001 0.001"/>
     </geometry>
   </collision>
@@ -153,5 +153,5 @@
     <origin xyz="0.117325 -0.101825 0.033" rpy="0 0 0"/>
     <geometry>
-      <mesh filename="file://$(find TankBot_description)/meshes/roda_dentada_v2__1__1.stl" scale="0.001 0.001 0.001"/>
+      <mesh filename="file://$(find tankbot_description)/meshes/roda_dentada_v2__1__1.stl" scale="0.001 0.001 0.001"/>
     </geometry>
     <material name="silver"/>
@@ -160,5 +160,5 @@
     <origin xyz="0.117325 -0.101825 0.033" rpy="0 0 0"/>
     <geometry>
-      <mesh filename="file://$(find TankBot_description)/meshes/roda_dentada_v2__1__1.stl" scale="0.001 0.001 0.001"/>
+      <mesh filename="file://$(find tankbot_description)/meshes/roda_dentada_v2__1__1.stl" scale="0.001 0.001 0.001"/>
     </geometry>
   </collision>
@@ -173,5 +173,5 @@
     <origin xyz="0.067305 -0.103825 0.069726" rpy="0 0 0"/>
     <geometry>
-      <mesh filename="file://$(find TankBot_description)/meshes/roda_lisa_v2__1__1.stl" scale="0.001 0.001 0.001"/>
+      <mesh filename="file://$(find tankbot_description)/meshes/roda_lisa_v2__1__1.stl" scale="0.001 0.001 0.001"/>
     </geometry>
     <material name="silver"/>
@@ -180,5 +180,5 @@
     <origin xyz="0.067305 -0.103825 0.069726" rpy="0 0 0"/>
     <geometry>
-      <mesh filename="file://$(find TankBot_description)/meshes/roda_lisa_v2__1__1.stl" scale="0.001 0.001 0.001"/>
+      <mesh filename="file://$(find tankbot_description)/meshes/roda_lisa_v2__1__1.stl" scale="0.001 0.001 0.001"/>
     </geometry>
   </collision>
@@ -193,5 +193,5 @@
     <origin xyz="0.022305 -0.103825 0.069726" rpy="0 0 0"/>
     <geometry>
-      <mesh filename="file://$(find TankBot_description)/meshes/roda_lisa_v2__7__1.stl" scale="0.001 0.001 0.001"/>
+      <mesh filename="file://$(find tankbot_description)/meshes/roda_lisa_v2__7__1.stl" scale="0.001 0.001 0.001"/>
     </geometry>
     <material name="silver"/>
@@ -200,5 +200,5 @@
     <origin xyz="0.022305 -0.103825 0.069726" rpy="0 0 0"/>
     <geometry>
-      <mesh filename="file://$(find TankBot_description)/meshes/roda_lisa_v2__7__1.stl" scale="0.001 0.001 0.001"/>
+      <mesh filename="file://$(find tankbot_description)/meshes/roda_lisa_v2__7__1.stl" scale="0.001 0.001 0.001"/>
     </geometry>
   </collision>
@@ -213,5 +213,5 @@
     <origin xyz="-0.022695 -0.103825 0.069726" rpy="0 0 0"/>
     <geometry>
-      <mesh filename="file://$(find TankBot_description)/meshes/roda_lisa_v2__9__1.stl" scale="0.001 0.001 0.001"/>
+      <mesh filename="file://$(find tankbot_description)/meshes/roda_lisa_v2__9__1.stl" scale="0.001 0.001 0.001"/>
     </geometry>
     <material name="silver"/>
@@ -220,5 +220,5 @@
     <origin xyz="-0.022695 -0.103825 0.069726" rpy="0 0 0"/>
     <geometry>
-      <mesh filename="file://$(find TankBot_description)/meshes/roda_lisa_v2__9__1.stl" scale="0.001 0.001 0.001"/>
+      <mesh filename="file://$(find tankbot_description)/meshes/roda_lisa_v2__9__1.stl" scale="0.001 0.001 0.001"/>
     </geometry>
   </collision>
@@ -233,5 +233,5 @@
     <origin xyz="-0.069695 -0.103825 0.069726" rpy="0 0 0"/>
     <geometry>
-      <mesh filename="file://$(find TankBot_description)/meshes/roda_lisa_v2__8__1.stl" scale="0.001 0.001 0.001"/>
+      <mesh filename="file://$(find tankbot_description)/meshes/roda_lisa_v2__8__1.stl" scale="0.001 0.001 0.001"/>
     </geometry>
     <material name="silver"/>
@@ -240,5 +240,5 @@
     <origin xyz="-0.069695 -0.103825 0.069726" rpy="0 0 0"/>
     <geometry>
-      <mesh filename="file://$(find TankBot_description)/meshes/roda_lisa_v2__8__1.stl" scale="0.001 0.001 0.001"/>
+      <mesh filename="file://$(find tankbot_description)/meshes/roda_lisa_v2__8__1.stl" scale="0.001 0.001 0.001"/>
     </geometry>
   </collision>
@@ -253,5 +253,5 @@
     <origin xyz="-0.120175 -0.101825 0.033" rpy="0 0 0"/>
     <geometry>
-      <mesh filename="file://$(find TankBot_description)/meshes/roda_lisa_v2_1.stl" scale="0.001 0.001 0.001"/>
+      <mesh filename="file://$(find tankbot_description)/meshes/roda_lisa_v2_1.stl" scale="0.001 0.001 0.001"/>
     </geometry>
     <material name="silver"/>
@@ -260,5 +260,5 @@
     <origin xyz="-0.120175 -0.101825 0.033" rpy="0 0 0"/>
     <geometry>
-      <mesh filename="file://$(find TankBot_description)/meshes/roda_lisa_v2_1.stl" scale="0.001 0.001 0.001"/>
+      <mesh filename="file://$(find tankbot_description)/meshes/roda_lisa_v2_1.stl" scale="0.001 0.001 0.001"/>
     </geometry>
   </collision>
